File: Analog_Line_Mixer_Stereo/Input_Module.sch (KiCad schematic (older format))
At the start: 11 parts, among them U2 LM833-N

Commit message: final commit for the night
Parts:
- C10, C7, C8, C9: footprint (none) -> Capacitors_SMD:C_1206
- R11, R12, R13, R14: footprint (none) -> Resistors_SMD:R_1206
Changed lines of the file:
@@
 F 0 "R23" V 1580 1800 50  0000 C CNN
 F 1 "47K" V 1500 1800 50  0000 C CNN
-F 2 "" V 1430 1800 50  0000 C CNN
+F 2 "Resistors_SMD:R_1206" V 1430 1800 50  0001 C CNN
 F 3 "" H 1500 1800 50  0000 C CNN
 	1    1500 1800
@@
 F 0 "R25" V 2230 1800 50  0000 C CNN
 F 1 "22K" V 2150 1800 50  0000 C CNN
-F 2 "" V 2080 1800 50  0000 C CNN
+F 2 "Resistors_SMD:R_1206" V 2080 1800 50  0001 C CNN
 F 3 "" H 2150 1800 50  0000 C CNN
 	1    2150 1800
@@
 F 0 "R26" V 2230 3550 50  0000 C CNN
 F 1 "22k" V 2150 3550 50  0000 C CNN
-F 2 "" V 2080 3550 50  0000 C CNN
+F 2 "Resistors_SMD:R_1206" V 2080 3550 50  0001 C CNN
 F 3 "" H 2150 3550 50  0000 C CNN
 	1    2150 3550
@@
 F 0 "R24" V 1580 3550 50  0000 C CNN
 F 1 "47K" V 1500 3550 50  0000 C CNN
-F 2 "" V 1430 3550 50  0000 C CNN
+F 2 "Resistors_SMD:R_1206" V 1430 3550 50  0001 C CNN
 F 3 "" H 1500 3550 50  0000 C CNN
 	1    1500 3550
@@
 F 0 "RV8" H 2760 3010 50  0000 C CNN
 F 1 "100K (Gain)" H 2890 2400 50  0000 C CNN
-F 2 "" H 2600 2700 50  0000 C CNN
+F 2 "" H 2600 2700 50  0001 C CNN
 F 3 "" H 2600 2700 50  0000 C CNN
 	1    2600 2700
@@
 F 0 "RV9" H 4460 2960 50  0000 C CNN
 F 1 "22K (Vol)" H 4590 2350 50  0000 C CNN
-F 2 "" H 4300 2650 50  0000 C CNN
+F 2 "" H 4300 2650 50  0001 C CNN
 F 3 "" H 4300 2650 50  0000 C CNN
 	1    4300 2650
@@
 F 0 "U5" H 3300 1700 60  0000 C CNN
 F 1 "LM833-N" H 3400 1800 60  0000 C CNN
-F 2 "" H 3400 1800 60  0000 C CNN
+F 2 "" H 3400 1800 60  0001 C CNN
 F 3 "" H 3400 1800 60  0000 C CNN
 	2    3350 1800
@@
 F 0 "U5" H 3250 3550 60  0000 C CNN
 F 1 "LM833-N" H 3350 3650 60  0000 C CNN
-F 2 "" H 3350 3650 60  0000 C CNN
+F 2 "" H 3350 3650 60  0001 C CNN
 F 3 "" H 3350 3650 60  0000 C CNN
 	1    3300 3650
@@
 F 0 "C19" H 1875 2300 50  0000 L CNN
 F 1 "47pF" H 1875 2100 50  0000 L CNN
-F 2 "" H 1888 2050 50  0000 C CNN
+F 2 "Capacitors_SMD:C_1206" H 1888 2050 50  0001 C CNN
 F 3 "" H 1850 2200 50  0000 C CNN
 	1    1850 2200
@@
 F 0 "C20" H 1875 3300 50  0000 L CNN
 F 1 "47pF" H 1875 3100 50  0000 L CNN
-F 2 "" H 1888 3050 50  0000 C CNN
+F 2 "Capacitors_SMD:C_1206" H 1888 3050 50  0001 C CNN
 F 3 "" H 1850 3200 50  0000 C CNN
 	1    1850 3200
@@
 F 0 "C22" H 3575 2450 50  0000 L CNN
 F 1 "100nF" H 3575 2250 50  0000 L CNN
-F 2 "" H 3588 2200 50  0000 C CNN
+F 2 "Capacitors_SMD:C_1206" H 3588 2200 50  0001 C CNN
 F 3 "" H 3550 2350 50  0000 C CNN
 	1    3550 2350
@@
 F 0 "C21" H 3575 1400 50  0000 L CNN
 F 1 "100nF" H 3575 1200 50  0000 L CNN
-F 2 "" H 3588 1150 50  0000 C CNN
+F 2 "Capacitors_SMD:C_1206" H 3588 1150 50  0001 C CNN
 F 3 "" H 3550 1300 50  0000 C CNN
 	1    3550 1300
