File: Analog_Line_Mixer_Stereo/Power_Reg.sch (KiCad schematic (older format))
At the start: 9 parts

Commit message: finalized schematic and started on board
Parts:
- removed D?: D, symbol D
- added D4: D_Schottky, Diodes_SMD:SOD-123, symbol D_Schottky
- C10, C11, C9: renamed from C?; footprint (none) -> Capacitors_SMD:C_1206
- L1: renamed from L?; footprint (none) -> Resistors_SMD:R_0805
- R16, R17, R18: renamed from R?; footprint (none) -> Resistors_SMD:R_1206
- U2: renamed from U?; footprint (none) -> TI-R-PDSO-G8:TI-LM2698-MUA08A
Connections:
- net GND: now also U2.4 (GND), U2.7 (FSLCT), U2.8 (NC_(GND))
- net Vout: now also D4.1 (K)
- net at L1.1, U2.5 (Vsw): now also D4.2 (A)
Changed lines of the file:
@@
 $EndDescr
 $Comp
-L LM2698 U?
+L LM2698 U2
 U 1 1 56B7CB94
 P 4750 2200
-F 0 "U?" H 4750 2150 60  0000 C CNN
+F 0 "U2" H 4750 2150 60  0000 C CNN
 F 1 "LM2698" H 4750 2300 60  0000 C CNN
-F 2 "" H 4750 2200 60  0000 C CNN
+F 2 "TI-R-PDSO-G8:TI-LM2698-MUA08A" H 4750 2200 60  0001 C CNN
 F 3 "" H 4750 2200 60  0000 C CNN
 	1    4750 2200
@@
 $EndComp
 $Comp
-L INDUCTOR L?
+L INDUCTOR L1
 U 1 1 56B7CBC4
 P 4150 2650
-F 0 "L?" V 4100 2650 50  0000 C CNN
+F 0 "L1" V 4100 2650 50  0000 C CNN
 F 1 "10uH" V 4250 2650 50  0000 C CNN
-F 2 "" H 4150 2650 50  0000 C CNN
+F 2 "Resistors_SMD:R_0805" H 4150 2650 50  0001 C CNN
 F 3 "" H 4150 2650 50  0000 C CNN
 	1    4150 2650
-	-1   0    0    1
-$EndComp
-$Comp
-L D D?
-U 1 1 56B7CC10
-P 4400 2950
-F 0 "D?" H 4400 3050 50  0000 C CNN
-F 1 "D" H 4400 2850 50  0000 C CNN
-F 2 "" H 4400 2950 50  0000 C CNN
-F 3 "" H 4400 2950 50  0000 C CNN
-	1    4400 2950
 	-1   0    0    1
 $EndComp
@@
 Vout
 $Comp
-L C C?
+L C C9
 U 1 1 56B7CC77
 P 3900 2650
-F 0 "C?" H 3925 2750 50  0000 L CNN
+F 0 "C9" H 3925 2750 50  0000 L CNN
 F 1 "22uF, 10V" V 3750 2500 50  0000 L CNN
-F 2 "" H 3938 2500 50  0000 C CNN
+F 2 "Capacitors_SMD:C_1206" H 3938 2500 50  0001 C CNN
 F 3 "" H 3900 2650 50  0000 C CNN
 	1    3900 2650
@@
 $EndComp
 $Comp
-L C C?
+L C C11
 U 1 1 56B7CCB3
 P 5250 3000
-F 0 "C?" H 5275 3100 50  0000 L CNN
+F 0 "C11" H 5275 3100 50  0000 L CNN
 F 1 "4.7nF" H 5275 2900 50  0000 L CNN
-F 2 "" H 5288 2850 50  0000 C CNN
+F 2 "Capacitors_SMD:C_1206" H 5288 2850 50  0001 C CNN
 F 3 "" H 5250 3000 50  0000 C CNN
 	1    5250 3000
@@
 $EndComp
 $Comp
-L R R?
+L R R16
 U 1 1 56B7CCD9
 P 5250 2600
-F 0 "R?" V 5330 2600 50  0000 C CNN
+F 0 "R16" V 5330 2600 50  0000 C CNN
 F 1 "24k9" V 5250 2600 50  0000 C CNN
-F 2 "" V 5180 2600 50  0000 C CNN
+F 2 "Resistors_SMD:R_1206" V 5180 2600 50  0001 C CNN
 F 3 "" H 5250 2600 50  0000 C CNN
 	1    5250 2600
@@
 $EndComp
 $Comp
-L R R?
+L R R18
 U 1 1 56B7CD3E
 P 5750 2250
-F 0 "R?" V 5830 2250 50  0000 C CNN
+F 0 "R18" V 5830 2250 50  0000 C CNN
 F 1 "30k1" V 5750 2250 50  0000 C CNN
-F 2 "" V 5680 2250 50  0000 C CNN
+F 2 "Resistors_SMD:R_1206" V 5680 2250 50  0001 C CNN
 F 3 "" H 5750 2250 50  0000 C CNN
 	1    5750 2250
@@
 $EndComp
 $Comp
-L R R?
+L R R17
 U 1 1 56B7CD73
 P 5500 2450
-F 0 "R?" V 5580 2450 50  0000 C CNN
+F 0 "R17" V 5580 2450 50  0000 C CNN
 F 1 "3k48" V 5500 2450 50  0000 C CNN
-F 2 "" V 5430 2450 50  0000 C CNN
+F 2 "Resistors_SMD:R_1206" V 5430 2450 50  0001 C CNN
 F 3 "" H 5500 2450 50  0000 C CNN
 	1    5500 2450
@@
 	5250 1950 5250 2050
 $Comp
-L GND #PWR?
-U 1 1 56B7D119
-P 5200 1950
-F 0 "#PWR?" H 5200 1700 50  0001 C CNN
-F 1 "GND" H 5200 1800 50  0000 C CNN
-F 2 "" H 5200 1950 50  0000 C CNN
-F 3 "" H 5200 1950 50  0000 C CNN
-	1    5200 1950
-	-1   0    0    1
-$EndComp
-$Comp
-L GND #PWR?
+L GND #PWR015
 U 1 1 56B7D189
 P 3900 3100
-F 0 "#PWR?" H 3900 2850 50  0001 C CNN
+F 0 "#PWR015" H 3900 2850 50  0001 C CNN
 F 1 "GND" H 3900 2950 50  0000 C CNN
 F 2 "" H 3900 3100 50  0000 C CNN
@@
 	5250 2750 5250 2850
 $Comp
-L GND #PWR?
+L GND #PWR016
 U 1 1 56B7D312
 P 5500 3150
-F 0 "#PWR?" H 5500 2900 50  0001 C CNN
+F 0 "#PWR016" H 5500 2900 50  0001 C CNN
 F 1 "GND" H 5500 3000 50  0000 C CNN
 F 2 "" H 5500 3150 50  0000 C CNN
@@
 	5250 3150 5500 3150
 $Comp
-L C C?
+L C C10
 U 1 1 56B7D3C6
 P 4650 2800
-F 0 "C?" H 4675 2900 50  0000 L CNN
+F 0 "C10" H 4675 2900 50  0000 L CNN
 F 1 "10uF" H 4675 2700 50  0000 L CNN
-F 2 "" H 4688 2650 50  0000 C CNN
+F 2 "Capacitors_SMD:C_1206" H 4688 2650 50  0001 C CNN
 F 3 "" H 4650 2800 50  0000 C CNN
 	1    4650 2800
@@
 $EndComp
 $Comp
-L GND #PWR?
+L GND #PWR017
 U 1 1 56B7D40A
 P 4650 2550
-F 0 "#PWR?" H 4650 2300 50  0001 C CNN
+F 0 "#PWR017" H 4650 2300 50  0001 C CNN
 F 1 "GND" H 4650 2400 50  0000 C CNN
 F 2 "" H 4650 2550 50  0000 C CNN
@@
 Text Label 6050 2250 0    60   ~ 0
 Vout
+$Comp
+L PWR_FLAG #FLG018
+U 1 1 56B80A26
+P 5250 2450
+F 0 "#FLG018" H 5250 2545 50  0001 C CNN
+F 1 "PWR_FLAG" H 5250 2630 50  0000 C CNN
+F 2 "" H 5250 2450 50  0000 C CNN
+F 3 "" H 5250 2450 50  0000 C CNN
+	1    5250 2450
+	0    -1   -1   0
+$EndComp
+$Comp
+L GND #PWR019
+U 1 1 56B829CC
+P 5250 1950
+F 0 "#PWR019" H 5250 1700 50  0001 C CNN
+F 1 "GND" H 5250 1800 50  0000 C CNN
+F 2 "" H 5250 1950 50  0000 C CNN
+F 3 "" H 5250 1950 50  0000 C CNN
+	1    5250 1950
+	-1   0    0    1
+$EndComp
+$Comp
+L D_Schottky D4
+U 1 1 56B86336
+P 4400 2950
+F 0 "D4" H 4400 3050 50  0000 C CNN
+F 1 "D_Schottky" H 4400 2850 50  0000 C CNN
+F 2 "Diodes_SMD:SOD-123" H 4400 2950 50  0001 C CNN
+F 3 "" H 4400 2950 50  0000 C CNN
+	1    4400 2950
+	-1   0    0    1
+$EndComp
 $EndSCHEMATC

Commit message: mostly finalized component placement, starting routing
Parts:
- U2: footprint TI-R-PDSO-G8:TI-LM2698-MUA08A -> texas:TI-LM2698-MUA08A
Changed lines of the file:
@@
 F 0 "U2" H 4750 2150 60  0000 C CNN
 F 1 "LM2698" H 4750 2300 60  0000 C CNN
-F 2 "TI-R-PDSO-G8:TI-LM2698-MUA08A" H 4750 2200 60  0001 C CNN
+F 2 "texas:TI-LM2698-MUA08A" H 4750 2200 60  0001 C CNN
 F 3 "" H 4750 2200 60  0000 C CNN
 	1    4750 2200
